File: BatCharger1S/BatCharger1S.kicad_sch (KiCad schematic)
At the start: 54 parts

Commit message: footprintAssigment
Parts:
- removed J?: 5V IN, symbol Connector:Conn_01x02_Socket
- removed J?: Switch, symbol Connector_Generic:Conn_01x02
- added J2: 5V IN, Connector_JST:JST_EH_B2B-EH-A_1x02_P2.50mm_Vertical, symbol Connector_Generic:Conn_01x02
- added J4: Switch, Connector_JST:JST_EH_B2B-EH-A_1x02_P2.50mm_Vertical, symbol Connector_Generic:Conn_01x02
- added J6: 3V3, Connector_JST:JST_EH_B2B-EH-A_1x02_P2.50mm_Vertical, symbol Connector_Generic:Conn_01x02
- added TP2: TestPoint, TestPoint:TestPoint_Pad_1.0x1.0mm, symbol Connector:TestPoint
- C1, C2, C3, C4, C5, C6, C7, C8, C9: renamed from C?; footprint (none) -> Capacitor_SMD:C_0603_1608Metric_Pad1.08x0.95mm_HandSolder
- D1, D2, D3: renamed from D?; footprint (none) -> LED_SMD:LED_0201_0603Metric_Pad0.64x0.40mm_HandSolder
- D4: renamed from D?; footprint (none) -> Diode_SMD:D_1206_3216Metric_Pad1.42x1.75mm_HandSolder
- D5: renamed from D?; value 6v -> 5v1; footprint (none) -> Diode_SMD:D_0603_1608Metric_Pad1.05x0.95mm_HandSolder
- FB1: renamed from FB?; footprint (none) -> Inductor_SMD:L_0402_1005Metric_Pad0.77x0.64mm_HandSolder
- J1: renamed from J?; footprint (none) -> Connector_USB:USB_C_Receptacle_Amphenol_12401548E4-2A
- J3, J5, J7: renamed from J?; footprint (none) -> Connector_JST:JST_EH_B2B-EH-A_1x02_P2.50mm_Vertical
- Q1: renamed from Q?; value PMOS -> SI2323DS; footprint (none) -> Package_TO_SOT_SMD:SOT-23-3
- Q2, Q3, Q4: renamed from Q?; value PMOS -> Si2323DS; footprint (none) -> Package_TO_SOT_SMD:SOT-23-3
- R1, R10, R11, R12, R13, R14, R15, R16, R17, R18, R19, R2, R3, R4, R5, R6, R7, R8, R9: renamed from R?; footprint (none) -> Resistor_SMD:R_0603_1608Metric_Pad0.98x0.95mm_HandSolder
- R20: renamed from R?; value 10k -> 100k; footprint (none) -> Resistor_SMD:R_0603_1608Metric_Pad0.98x0.95mm_HandSolder
- TH1: renamed from TH?; footprint (none) -> Resistor_SMD:R_0603_1608Metric_Pad0.98x0.95mm_HandSolder
- TP1, TP3, TP4, TP5: renamed from TP?; footprint (none) -> TestPoint:TestPoint_Pad_1.0x1.0mm
- U2: renamed from U?; footprint 21-0168E_T822-3_MXM -> Package_DFN_QFN:TDFN-8-1EP_2x2mm_P0.5mm_EP0.8x1.2mm
- U3: renamed from U?; footprint MSOP10_MC_MCH -> Package_SO:MSOP-10-1EP_3x3mm_P0.5mm_EP1.68x1.88mm
- gave numbers to parts that had none: 2
Connections:
- net +3V3: now also J6.1 (Pin_1)
- net +5V: now also Q2.1 (D), J2.1 (Pin_1); no longer Q2.3 (S)
- net GND: now also J2.2 (Pin_2), J6.2 (Pin_2)
- net VBUS: now also Q1.1 (D); no longer Q1.3 (S)
- net VCC: now also J4.1 (Pin_1); no longer D4.1 (K), Q3.3 (S)
- net VDC: now also Q1.3 (S), Q2.3 (S), TP2.1; no longer Q1.1 (D), Q2.1 (D)
- new net: D4.1 (K), J4.2 (Pin_2), Q3.3 (S)
Other:
- note added: "- Load Sharing (PSU permiting Charge and use System as same time) - USB-C or 5V DC Input (No OV Protection) - Power MUX for Dual Input Protection - I2C Fuel Gauge (Remive 0R resistor to disable) - Charging Status LEDs"
- note added: "1S Li-Ion/Phosphate Charger"
- note added: "1S Li-Ion/Po Battery Charger Module"
- note removed: "Charger"
- note removed: "Load Sharing"
- note removed: "Short Disable Reg"
- company: (none) -> WRSROBOTICS
- title: (none) -> 1S Li-Ion Charger
- moved on the sheet: C1, C2, C3, C4, C5, C7, D5, FB1, J1, J3, J5, Q1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

Commit message: bom
Parts:
- added H1, H2, H3, H4: MountingHole, symbol Mechanical:MountingHole
- J2: value 5V IN -> 01x02
- J3: value USB2.0 -> 01x02
- J4: value Switch -> 01x02
- J5: footprint Connector_JST:JST_EH_B2B-EH-A_1x02_P2.50mm_Vertical -> Connector_JST:JST_EH_B3B-EH-A_1x03_P2.50mm_Vertical
- J6: value 3V3 -> 01x02
- J7: value BAT -> 01x02
- Q1: value SI2323DS -> Si2323DS
Changed lines of the file:
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@@
+    )
+  )
+  (symbol (lib_id "Mechanical:MountingHole") (at 19.05 121.92 0) (unit 1)
+    (in_bom yes) (on_board yes) (dnp no) (fields_autoplaced)
+    (property "Reference" "H2" (at 21.59 120.65 0)
+      (effects (font (size 1.27 1.27)) (justify left))
+    )
+    (property "Value" "MountingHole" (at 21.59 123.19 0)
+      (effects (font (size 1.27 1.27)) (justify left))
+    )
+    (property "Footprint" "" (at 19.05 121.92 0)
+      (effects (font (size 1.27 1.27)) hide)
+    )
+    (property "Datasheet" "~" (at 19.05 121.92 0)
+      (effects (font (size 1.27 1.27)) hide)
+    )
+    (instances
+      (project "BatCharger1S"
+        (path "/cb4dccd2-31cd-48d8-8ae1-ec97ee332fde"
+          (reference "H2") (unit 1)
+        )
+      )
     )
   )
@@
       (effects (font (size 1.27 1.27)) (justify left))
     )
-    (property "Value" "USB2.0" (at 104.14 52.07 0)
+    (property "Value" "01x02" (at 104.14 52.07 0)
       (effects (font (size 1.27 1.27)) (justify left))
     )
@@
     )
   )
+  (symbol (lib_id "Mechanical:MountingHole") (at 19.05 128.27 0) (unit 1)
+    (in_bom yes) (on_board yes) (dnp no) (fields_autoplaced)
+    (property "Reference" "H3" (at 21.59 127 0)
+      (effects (font (size 1.27 1.27)) (justify left))
+    )
+    (property "Value" "MountingHole" (at 21.59 129.54 0)
+      (effects (font (size 1.27 1.27)) (justify left))
+    )
+    (property "Footprint" "" (at 19.05 128.27 0)
+      (effects (font (size 1.27 1.27)) hide)
+    )
+    (property "Datasheet" "~" (at 19.05 128.27 0)
+      (effects (font (size 1.27 1.27)) hide)
+    )
+    (instances
+      (project "BatCharger1S"
+        (path "/cb4dccd2-31cd-48d8-8ae1-ec97ee332fde"
+          (reference "H3") (unit 1)
+        )
+      )
+    )
+  )
   (symbol (lib_id "power:GND") (at 59.69 41.91 0) (unit 1)
     (in_bom yes) (on_board yes) (dnp no) (fields_autoplaced)
@@
       (effects (font (size 1.27 1.27)) (justify left))
     )
-    (property "Value" "BAT" (at 276.86 33.02 0)
+    (property "Value" "01x02" (at 276.86 33.02 0)
       (effects (font (size 1.27 1.27)) (justify left))
     )
@@
       (effects (font (size 1.27 1.27)) (justify left))
     )
-    (property "Value" "Switch" (at 196.85 95.25 90)
+    (property "Value" "01x02" (at 196.85 95.25 90)
       (effects (font (size 1.27 1.27)) (justify left))
     )
@@
       (effects (font (size 1.27 1.27)))
     )
-    (property "Value" "SI2323DS" (at 100.33 68.58 90)
+    (property "Value" "Si2323DS" (at 100.33 68.58 90)
       (effects (font (size 1.27 1.27)))
     )
@@
       (effects (font (size 1.27 1.27)) (justify left))
     )
-    (property "Value" "5V IN" (at 68.58 100.33 0)
+    (property "Value" "01x02" (at 68.58 100.33 0)
       (effects (font (size 1.27 1.27)) (justify left))
     )
@@
     )
   )
+  (symbol (lib_id "Mechanical:MountingHole") (at 19.05 134.62 0) (unit 1)
+    (in_bom yes) (on_board yes) (dnp no) (fields_autoplaced)
+    (property "Reference" "H4" (at 21.59 133.35 0)
+      (effects (font (size 1.27 1.27)) (justify left))
+    )
+    (property "Value" "MountingHole" (at 21.59 135.89 0)
+      (effects (font (size 1.27 1.27)) (justify left))
+    )
+    (property "Footprint" "" (at 19.05 134.62 0)
+      (effects (font (size 1.27 1.27)) hide)
+    )
+    (property "Datasheet" "~" (at 19.05 134.62 0)
+      (effects (font (size 1.27 1.27)) hide)
+    )
+    (instances
+      (project "BatCharger1S"
+        (path "/cb4dccd2-31cd-48d8-8ae1-ec97ee332fde"
+          (reference "H4") (unit 1)
+        )
+      )
+    )
+  )
   (symbol (lib_id "power:GND") (at 224.79 133.35 0) (unit 1)
     (in_bom yes) (on_board yes) (dnp no) (fields_autoplaced)
@@
       (effects (font (size 1.27 1.27)) (justify left))
     )
-    (property "Value" "3V3" (at 256.54 87.63 0)
+    (property "Value" "01x02" (at 256.54 87.63 0)
       (effects (font (size 1.27 1.27)) (justify left))
     )
@@
       (effects (font (size 1.27 1.27)) (justify left) hide)
     )
-    (property "Footprint" "Connector_JST:JST_EH_B2B-EH-A_1x02_P2.50mm_Vertical" (at 252.73 125.73 0)
+    (property "Footprint" "Connector_JST:JST_EH_B3B-EH-A_1x03_P2.50mm_Vertical" (at 252.73 125.73 0)
       (effects (font (size 1.27 1.27)) hide)
     )
@@
         )
       )
+    )
+  )
+  (symbol (lib_id "Mechanical:MountingHole") (at 19.05 115.57 0) (unit 1)
+    (in_bom yes) (on_board yes) (dnp no) (fields_autoplaced)
+    (property "Reference" "H1" (at 21.59 114.3 0)
+      (effects (font (size 1.27 1.27)) (justify left))
+    )
+    (property "Value" "MountingHole" (at 21.59 116.84 0)
+      (effects (font (size 1.27 1.27)) (justify left))
+    )
+    (property "Footprint" "" (at 19.05 115.57 0)
+      (effects (font (size 1.27 1.27)) hide)
+    )
+    (property "Datasheet" "~" (at 19.05 115.57 0)
+      (effects (font (size 1.27 1.27)) hide)
+    )
+    (instances
+      (project "BatCharger1S"
+        (path "/cb4dccd2-31cd-48d8-8ae1-ec97ee332fde"
+          (reference "H1") (unit 1)
+        )
+      )

Commit message: PCBv0.1
Parts:
- removed D5: 5v1, Diode_SMD:D_0603_1608Metric_Pad1.05x0.95mm_HandSolder, symbol Device:D_Zener
- removed J6: 01x02, Connector_JST:JST_EH_B2B-EH-A_1x02_P2.50mm_Vertical, symbol Connector_Generic:Conn_01x02
- removed TH1: NTC, Resistor_SMD:R_0603_1608Metric_Pad0.98x0.95mm_HandSolder, symbol Device:Thermistor_NTC
- added J5: 01x02, Connector_JST:JST_EH_B2B-EH-A_1x02_P2.50mm_Vertical, symbol Connector_Generic:Conn_01x02
- C1, C4: value 4u7 -> 10u
- D3: value Yellow -> Red
- FB1: value BK603HS330-T -> 100 @ 100MHz
- H1, H2, H3, H4: footprint (none) -> MountingHole:MountingHole_2.2mm_M2
- TP1, TP2, TP3, TP4, TP5: footprint TestPoint:TestPoint_Pad_1.0x1.0mm -> TestPoint:TestPoint_Pad_D1.0mm
- renumbered J5 to J6
Connections:
- net +3V3: now also J5.2 (Pin_2)
- net +BATT: no longer C5.1
- net CON_USB_N: now also U1.1 (I/O1); no longer U1.6 (I/O1)
- net CON_USB_P: now also U1.6 (I/O1); no longer U1.1 (I/O1)
- net GND: now also J5.1 (Pin_1)
- net SCl: now also J6.2 (Pin_2); no longer J6.3 (Pin_3)
- net SDA: now also J6.3 (Pin_3); no longer J6.2 (Pin_2)
- net USB_N: now also U1.3 (I/O2); no longer U1.4 (I/O2)
- net USB_P: now also U1.4 (I/O2); no longer U1.3 (I/O2)
- net vBatSense: now also C5.1
- net VBUS_IN: now reaches C2.1, C3.1, FB1.1, J1.A4 (VBUS), J1.A9 (VBUS), J1.B4 (VBUS), J1.B9 (VBUS), U1.5 (VBUS)
- net pwrSwitch: now reaches D4.1 (K), J4.2 (Pin_2), Q3.3 (S)
Other:
- note added: "DC Input 5V"
- note added: "Switch Connector"
- note added: "USB Connector"
- moved on the sheet: C5, J7, R18, R19, R20

Commit message: v2Layout
Parts:
- removed C1: 10u, Capacitor_SMD:C_0603_1608Metric_Pad1.08x0.95mm_HandSolder, symbol Device:C_Small
- removed C3: 1u, Capacitor_SMD:C_0603_1608Metric_Pad1.08x0.95mm_HandSolder, symbol Device:C_Small
- removed FB1: 100 @ 100MHz, Inductor_SMD:L_0402_1005Metric_Pad0.77x0.64mm_HandSolder, symbol Device:FerriteBead_Small
- removed J1: USB_C_Receptacle, Connector_USB:USB_C_Receptacle_Amphenol_12401548E4-2A, symbol Connector:USB_C_Receptacle
- removed J5: 01x02, Connector_JST:JST_EH_B2B-EH-A_1x02_P2.50mm_Vertical, symbol Connector_Generic:Conn_01x02
- removed J6: Conn_01x03, Connector_JST:JST_EH_B3B-EH-A_1x03_P2.50mm_Vertical, symbol Connector_Generic:Conn_01x03
- removed R1: 1M, Resistor_SMD:R_0603_1608Metric_Pad0.98x0.95mm_HandSolder, symbol Device:R_Small
- added C2: 10u, Capacitor_SMD:C_0805_2012Metric_Pad1.18x1.45mm_HandSolder, symbol Device:C_Small
- added J1: TYPE-C-31-M-12, Connector_USB:TYPE-C-31-M-12, symbol Connector:TYPE-C-31-M-12
- added J5: Conn_01x03, Connector_JST:JST_EH_B3B-EH-A_1x03_P2.50mm_Vertical, symbol Connector_Generic:Conn_01x03
- added J6: 01x02, Connector_JST:JST_EH_B2B-EH-A_1x02_P2.50mm_Vertical, symbol Connector_Generic:Conn_01x02
- added Q1: Si2323DS, Package_TO_SOT_SMD:SOT-23-3, symbol Simulation_SPICE:PMOS
- added R4: 10k, Resistor_SMD:R_0603_1608Metric_Pad0.98x0.95mm_HandSolder, symbol Device:R_Small
- J4: footprint Connector_JST:JST_EH_B2B-EH-A_1x02_P2.50mm_Vertical -> Connector_PinHeader_2.54mm:PinHeader_1x02_P2.54mm_Vertical
- U3: footprint Package_SO:MSOP-10-1EP_3x3mm_P0.5mm_EP1.68x1.88mm -> Package_SO:MSOP-10_3x3mm_P0.5mm
- renumbered C2 to C3, Q1 to Q2, Q2 to Q3, Q3 to Q4, Q4 to Q5, R9 to R10, R10 to R11, R11 to R12, R12 to R13, R13 to R14, R14 to R15, R15 to R16, R16 to R17, R17 to R18, R18 to R19, R19 to R20, R20 to R21, R4 to R5, R5 to R6, R6 to R7, R7 to R8, R8 to R9
Connections:
- net VBUS_IN is gone; now on net VBUS: C3.1, U1.5 (VBUS)
- net +3V3: now also J6.2 (Pin_2)
- net +5V: now also C2.1, Q1.3 (S); no longer J2.1 (Pin_1)
- net Alert: now also J5.1 (Pin_1)
- net CON_USB_N: now also J1.A7 (D-)
- net CON_USB_P: now also J1.A6 (D+)
- net GND: now also J2.1 (Pin_1), C2.2, J1.A1 (GND), J1.A12 (GND), J1.B1 (GND), J1.B12 (GND), J1.S1 (SHIELD), J6.1 (Pin_1), R4.2; no longer J2.2 (Pin_2)
- net SCl: now also J5.3 (Pin_3)
- net SDA: now also J5.2 (Pin_2)
- net VBUS: now also J1.A4 (VBUS), J1.A9 (VBUS), J1.B4 (VBUS), J1.B9 (VBUS)
- net at R3.1: now also J1.A5 (CC)
- net at R2.1: now also J1.B5 (VCONN)
- new net: J2.2 (Pin_2), Q1.1 (D)
- new net: Q1.2 (G), R4.1
- no-connect marks 11 -> 1
Other:
- moved on the sheet: TP1
